File: v01/tryptris_pcb.sch (KiCad schematic (older format))
At the start: 131 parts, among them J1 USB_C_Receptacle_USB2.0, J2 I2C-L, J3 I2C-R, SW1 Reset, U1 ATmega32U4-AU, U2 MCP23017_SO, Y1 16Mhz

Commit message: Swap TRRS connectors out for USBC
I have never been a big fan of TRRS and using USBC should be ok as I'm
keeping the 5V and GND pins the same as with USB.
Parts:
- removed J2: I2C-L, Connector_Audio:Jack_3.5mm_PJ320E_Horizontal, symbol Connector:AudioJack4
- removed J3: I2C-R, Connector_Audio:Jack_3.5mm_PJ320E_Horizontal, symbol Connector:AudioJack4
- removed R10, R9: 4.7k, Resistor_SMD:R_0805_2012Metric, symbol Device:R_Small
- added J2: I2C-L, Type-C:USB_C_GCT_USB4085, symbol Connector:USB_C_Receptacle_USB2.0
- added J3: I2C-R, Type-C:USB_C_GCT_USB4085, symbol Connector:USB_C_Receptacle_USB2.0
- added R6, R7: 4.7k, Resistor_SMD:R_0805_2012Metric, symbol Device:R_Small
Connections:
- wire segments 261 -> 277
