File: v01/tryptris_pcb.sch (KiCad schematic (older format))
At the start: 131 parts, among them J1 USB_C_Receptacle_USB2.0, J2 I2C-L, J3 I2C-R, SW1 Reset, U1 ATmega32U4-AU, U2 MCP23017_SO, Y1 16Mhz

Commit message: Get RGB matrix roughed in.
Other:
- note added: "IO Expander\n\naddress:\n100 + A2 + A1 + A0 + rw\n100000rw"
- note removed: "IO Expander"
Changed lines of the file:
@@
 Col5
 Text Notes 2800 6200 0    50   ~ 0
-IO Expander
+IO Expander\n\naddress:\n100 + A2 + A1 + A0 + rw\n100000rw
 Wire Wire Line
 	9000 6950 8600 6950
