File: v01/rgb matrix.sch (KiCad schematic (older format))
At the start: 66 parts, among them U4 IS31FL3731-SA

Commit message: Get RGB matrix roughed in.
Parts:
- removed C? (x2): 1uF, symbol Device:C_Small
- removed C?: 0.1uF, symbol Device:C_Small
- removed C?: C_Small, symbol Device:C_Small
- removed D? (x27): 6028 LED, symbol Device:LED_BRAG
- removed R?: 100K, symbol Device:R_Small
- removed R?: R_Small, symbol Device:R_Small
- removed R?: 20K, symbol Device:R_Small
- removed U4, U?: IS31FL3731-SA, Package_SO:SSOP-28_5.3x10.2mm_P0.65mm, symbol Driver_LED:IS31FL3731-SA
- added C? (x6): 01.uF, symbol Device:C_Small
- added C? (x8): 0.47uF, symbol Device:C_Small
- added D? (x27): 6028 LED, symbol Device:LED_BRAG
- added R? (x2): 100K, symbol Device:R_Small
- added R?: 20K, symbol Device:R_Small
- added U? (x2): IS31FL3733-TQ, Package_QFP:TQFP-48-1EP_7x7mm_P0.5mm_EP5x5mm, symbol Driver_LED:IS31FL3733-TQ
- R?: value 4.7K -> 100K
Connections:
- net Left-CB4 is gone; now on net Left-SW12: D?.1 (BK), D?.1 (BK), D?.1 (BK)
- net Left-CB5 is gone; now on net Left-SW11: D?.2 (RK)
- net Left-CB6 is gone; now on net Left-SW10: D?.4 (GK)
- net Left-CB7 is gone; now on net Left-SW12: D?.1 (BK)
- net +5V: now also C?.1, C?.1, C?.1, C?.1, C?.2, C?.2, U?.20 (PVCC), U?.29 (PVCC), U?.37 (AVCC), U?.38 (DVCC); no longer R?.2, R?.2
- net GND: now also R?.2, R?.2, C?.1, C?.1, C?.1, C?.1, C?.1, C?.1, C?.2, C?.2, C?.2, C?.2, C?.2, C?.2, C?.2, C?.2, R?.2, R?.2, R?.2, U?.12 (PGND), U?.12 (PGND), U?.34 (AGND), U?.34 (AGND), U?.43 (ADDR1), U?.44 (ADDR2), U?.44 (ADDR2), U?.48 (GND), U?.48 (GND), U?.49 (GND), U?.49 (GND), U?.5 (PGND), U?.5 (PGND)
- net SCL-L: now also U?.42 (SCL), U?.42 (SCL), U?.43 (ADDR1)
- net SDA-L: now also U?.41 (SDA), U?.41 (SDA)
- net VBUS: now also C?.2, C?.2, U?.39 (VIO), U?.39 (VIO)
- net at R?.1: now also U?.46 (~SDB)
- net at R?.1: now also U?.47 (IICRST)
- net at R?.1: now also U?.35 (RSET)
- net Left-SW9: now reaches D?.1 (BK)
- net Left-SW9: now also D?.1 (BK), D?.1 (BK), D?.1 (BK), D?.1 (BK), D?.1 (BK), U?.11 (SW9)
- net Left-SW8: now reaches D?.2 (RK)
- net Left-SW8: now also D?.2 (RK), D?.2 (RK), D?.2 (RK), D?.2 (RK), D?.2 (RK), U?.10 (SW8)
- net Left-CS1: now reaches D?.3 (A)
- net Left-CS1: now also D?.3 (A), D?.3 (A), D?.3 (A), U?.16 (CS1)
- net Left-SW7: now reaches D?.4 (GK)
- net Left-SW7: now also D?.4 (GK), D?.4 (GK), D?.4 (GK), D?.4 (GK), D?.4 (GK), U?.9 (SW7)
- net Left-SW6: now reaches D?.1 (BK)
- net Left-SW6: now also D?.1 (BK), D?.1 (BK), D?.1 (BK), D?.1 (BK), D?.1 (BK), U?.8 (SW6)
- net Left-SW5: now reaches D?.2 (RK)
- net Left-SW5: now also D?.2 (RK), D?.2 (RK), D?.2 (RK), D?.2 (RK), D?.2 (RK), U?.7 (SW5)
- net Left-SW4: now reaches D?.4 (GK)
- net Left-SW4: now also D?.4 (GK), D?.4 (GK), D?.4 (GK), D?.4 (GK), D?.4 (GK), U?.6 (SW4)
- net Left-SW3: now reaches D?.1 (BK)
- net Left-SW3: now also D?.1 (BK), D?.1 (BK), D?.1 (BK), D?.1 (BK), D?.1 (BK), D?.1 (BK), D?.1 (BK), D?.1 (BK), D?.1 (BK), D?.1 (BK), D?.1 (BK), U?.4 (SW3)
- net Left-SW2: now reaches D?.2 (RK)
- net Left-SW2: now also D?.2 (RK), D?.2 (RK), D?.2 (RK), D?.2 (RK), D?.2 (RK), D?.2 (RK), D?.2 (RK), D?.2 (RK), D?.2 (RK), D?.2 (RK), D?.2 (RK), U?.3 (SW2)
- net Left-SW1: now reaches D?.4 (GK)
- net Left-SW1: now also D?.4 (GK), D?.4 (GK), D?.4 (GK), D?.4 (GK), D?.4 (GK), D?.4 (GK), D?.4 (GK), D?.4 (GK), D?.4 (GK), D?.4 (GK), D?.4 (GK), U?.2 (SW1)
- net Left-CS2: now reaches D?.3 (A)
- net Left-CS2: now also D?.3 (A), D?.3 (A), D?.3 (A), U?.17 (CS2)
- net Left-CS3: now reaches D?.3 (A)
- net Left-CS3: now also D?.3 (A), D?.3 (A), D?.3 (A), U?.18 (CS3)
- net Left-CS4: now reaches D?.3 (A)
- net Left-CS4: now also D?.3 (A), D?.3 (A), D?.3 (A), U?.19 (CS4)
- net Left-CS5: now reaches D?.3 (A)
- net Left-CS5: now also D?.3 (A), D?.3 (A), D?.3 (A), U?.21 (CS5)
- net Left-CS6: now reaches D?.3 (A)
- net Left-CS6: now also D?.3 (A), D?.3 (A), D?.3 (A), U?.22 (CS6)
- net Left-CS7: now reaches D?.3 (A)
- net Left-CS7: now also U?.23 (CS7)
- net Left-CS8: now reaches D?.3 (A)
- net Left-CS8: now also U?.24 (CS8)
- net Left-CS9: now reaches D?.3 (A)
- net Left-CS9: now also U?.25 (CS9)
- net Left-CA5 renamed Left-SW11
- net Left-SW11: now also D?.2 (RK), D?.2 (RK), D?.2 (RK), U?.14 (SW11)
- net Left-CA6 renamed Left-SW10
- net Left-SW10: now also D?.4 (GK), D?.4 (GK), D?.4 (GK), U?.13 (SW10)
- net Left-CA7 renamed Left-SW12
- net Left-SW12: now also U?.15 (SW12)
- removed net Left-CB1: D?.2 (RK), D?.2 (RK), D?.3 (A), D?.3 (A)
- removed net Left-CB2: D?.2 (RK), D?.3 (A), D?.3 (A), D?.4 (GK)
- removed net Left-CB3: D?.3 (A), D?.3 (A), D?.4 (GK), D?.4 (GK)
- new net: R?.1, U?.46 (~SDB)
- new net: R?.1, U?.47 (IICRST)
- new net: R?.1, U?.35 (RSET)
- new net: C?.1, C?.1, U?.20 (PVCC)
- new net: C?.1, C?.2, U?.29 (PVCC)
- new net: C?.1, C?.2, U?.37 (AVCC), U?.38 (DVCC)
- new net Right-CS1: D?.3 (A), D?.3 (A), D?.3 (A), D?.3 (A), U?.16 (CS1)
- new net Right-CS2: D?.3 (A), D?.3 (A), D?.3 (A), D?.3 (A), U?.17 (CS2)
- new net Right-CS3: D?.3 (A), D?.3 (A), D?.3 (A), D?.3 (A), U?.18 (CS3)
- new net Right-CS4: D?.3 (A), D?.3 (A), D?.3 (A), D?.3 (A), U?.19 (CS4)
- new net Right-CS5: D?.3 (A), D?.3 (A), D?.3 (A), D?.3 (A), U?.21 (CS5)
- new net Right-CS6: D?.3 (A), D?.3 (A), D?.3 (A), D?.3 (A), U?.22 (CS6)
- new net Right-CS7: D?.3 (A), U?.23 (CS7)
- new net Right-CS8: D?.3 (A), U?.24 (CS8)
- new net Right-CS9: D?.3 (A), U?.25 (CS9)
- new net Right-SW1: D?.4 (GK), D?.4 (GK), D?.4 (GK), D?.4 (GK), D?.4 (GK), D?.4 (GK), U?.2 (SW1)
- new net Right-SW10: D?.4 (GK), D?.4 (GK), D?.4 (GK), D?.4 (GK), D?.4 (GK), D?.4 (GK), U?.13 (SW10)
- new net Right-SW11: D?.2 (RK), D?.2 (RK), D?.2 (RK), D?.2 (RK), D?.2 (RK), D?.2 (RK), U?.14 (SW11)
- new net Right-SW12: D?.1 (BK), D?.1 (BK), D?.1 (BK), D?.1 (BK), D?.1 (BK), D?.1 (BK), U?.15 (SW12)
- new net Right-SW2: D?.2 (RK), D?.2 (RK), D?.2 (RK), D?.2 (RK), D?.2 (RK), D?.2 (RK), U?.3 (SW2)
- new net Right-SW3: D?.1 (BK), D?.1 (BK), D?.1 (BK), D?.1 (BK), D?.1 (BK), D?.1 (BK), U?.4 (SW3)
- new net Right-SW4: D?.4 (GK), D?.4 (GK), D?.4 (GK), D?.4 (GK), D?.4 (GK), D?.4 (GK), U?.6 (SW4)
- new net Right-SW5: D?.2 (RK), D?.2 (RK), D?.2 (RK), D?.2 (RK), D?.2 (RK), D?.2 (RK), U?.7 (SW5)
- new net Right-SW6: D?.1 (BK), D?.1 (BK), D?.1 (BK), D?.1 (BK), D?.1 (BK), D?.1 (BK), U?.8 (SW6)
- new net Right-SW7: D?.4 (GK), D?.4 (GK), D?.4 (GK), D?.4 (GK), D?.4 (GK), D?.4 (GK), U?.9 (SW7)
- new net Right-SW8: D?.2 (RK), D?.2 (RK), D?.2 (RK), D?.2 (RK), D?.2 (RK), D?.2 (RK), U?.10 (SW8)
- new net Right-SW9: D?.1 (BK), D?.1 (BK), D?.1 (BK), D?.1 (BK), D?.1 (BK), D?.1 (BK), U?.11 (SW9)
- no-connect marks 4 -> 7
Other:
- note added: "Left side\naddress:\n101 + A1 + A2 + R/W\n1010000rw"
- note added: "Right side\naddress:\n101 + A1 + A2 +R/W\n1010001rw"
- note removed: "Left side\naddress:\n11101 + AD + R/W\n1110100rw"
- note removed: "Right side\naddress:\n11101 + AD +R/W\n1110101rw"
- moved on the sheet: D?, R?

Commit message: Fix ERC errors.
Parts:
- gave numbers to parts that had none: 76
Connections:
- net GND: no longer C10.2, C14.2, C15.2, C16.1, C20.1, C8.1, C9.2, R10.2, R13.2, R9.2, U3.12 (PGND), U3.34 (AGND), U3.44 (ADDR2), U3.48 (GND), U3.49 (GND), U3.5 (PGND)
- net VBUS: now also C10.1, C14.1, C15.1, C16.2, C8.2, C9.1, U3.20 (PVCC), U3.29 (PVCC), U3.37 (AVCC), U3.38 (DVCC)
- new net VSS: C10.2, C14.2, C15.2, C16.1, C20.1, C8.1, C9.2, R10.2, R13.2, R9.2, U3.12 (PGND), U3.34 (AGND), U3.44 (ADDR2), U3.48 (GND), U3.49 (GND), U3.5 (PGND)
- no-connect marks 7 -> 19
Other:
- moved on the sheet: C10, C14, C15, C16, C20, C8, C9, R10, R13, R9, U3
