File: v01/bling-case/ursaminor_pcb.kicad_pcb (KiCad board)
At the start: 2 copper layers, 298.6 x 118.1 mm, 209 parts, among them J1 USB_C_Receptacle_USB2.0, J2 I2C-L, J3 I2C-R, J4 AVR-ISP-6, SW1 Reset, U1 ATmega32U4-AU, U2 MCP23017_SO, U3 IS31FL3733-TQ, U4 IS31FL3733-TQ, U5 PRTR5V0U2X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

Commit message: Finished routing and via stitching the gnd planes together.
Routing:
- net Right-SW12: track 108.7 -> 193.9 mm, vias 0 -> 2
- net Right-SW11: track 129.5 -> 214.5 mm, vias 10 -> 12
- net Right-SW10: track 138.6 -> 220.2 mm, vias 0 -> 2
- net VSS: track 59.9 -> 69.2 mm, vias 59 -> 104
- net Row2-R: track 141.6 -> 145.3 mm
- net Row1-R: track 162.6 -> 166.1 mm
- net VBUS: track 184.6 -> 187.3 mm
- net Right-CS1: track 151.0 -> 153.4 mm
- net Right-CS5: track 109.4 -> 111.4 mm
- net Col8: track 141.0 -> 142.7 mm
- net Col9: track 133.6 -> 134.9 mm
- net Right-SW6: track 150.5 -> 151.4 mm
- net Col11: track 212.6 -> 213.5 mm
- net Col7: track 183.9 -> 184.7 mm
- net Right-CS6: track 135.7 -> 136.3 mm
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
Commit message: Fix DRC errors.
Routing:
- net Col2: track 145.9 -> 142.1 mm
- net Row1-L: track 172.1 -> 174.4 mm
- net SCL-R: track 91.9 -> 93.6 mm
- net GND: track 145.9 -> 147.4 mm, vias 102 -> 106
- net Net-(J4-Pad5): track 148.7 -> 149.5 mm
- net D+: track 80.4 -> 81.0 mm
- net VSS: vias 104 -> 105

Commit message: Reduce area used and fix outline and DRC
Parts:
- added REF**: breakaway-mousebites, Keebio-Parts:breakaway-mousebites, F.Cu at (159.2, 96.2)
- added REF**: breakaway-mousebites, Keebio-Parts:breakaway-mousebites, F.Cu at (163.0, 96.2)
- added REF**: breakaway-mousebites, Keebio-Parts:breakaway-mousebites, F.Cu at (163.0, 34.0)
- added REF**: breakaway-mousebites, Keebio-Parts:breakaway-mousebites, F.Cu at (159.2, 34.0)
- moved C15 154.1 mm to (113.1, 97.0)
- moved C9 154.1 mm to (117.8, 97.0)
- moved D100 154.1 mm to (110.9, 86.2)
- moved D106 154.1 mm to (26.1, 120.5)
- moved D108 154.1 mm to (66.8, 107.7)
- moved D28 154.1 mm to (49.2, 39.6)
- moved D29 154.1 mm to (68.2, 37.2)
- moved D32 154.1 mm to (125.3, 44.4)
- moved D33 154.1 mm to (144.3, 44.4)
- moved D35 154.1 mm to (68.2, 56.2)
- moved D38 154.1 mm to (125.3, 63.4)
- moved D40 154.1 mm to (49.2, 77.6)
- moved D41 154.1 mm to (68.2, 75.2)
- moved D45 154.1 mm to (144.2, 82.4)
- moved D47 154.1 mm to (64.9, 91.0)
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Other:
- board size 298.6 x 118.1 mm -> 294.3 x 118.1 mm

Commit message: Add silkscreen to top and adjust bottom silkscreen.
Parts:
- added G***: LOGO, v01:v2-board-top-silkscreen-right, F.Cu at (87.1, 148.0)
- added G***: LOGO, v01:v2-board-top-silkscreen, F.Cu at (234.5, 148.0)
- turned D52 to 34.5 degrees
Routing:
- net Row4-R: track 55.2 -> 58.2 mm
- net Net-(D52-Pad2): track 12.4 -> 13.1 mm
Other:
- board text added: "markstory/ursa-minor : rev02"
- board text removed: "Ursa Minor rev01 : markstory"
